File: schematics/gate_driver.kicad_sch (KiCad schematic)
At the start: 13 parts, among them T2 P0584NL, U10 VO2611, U11 TC4420

Commit message: Small schematic fixes
Parts:
- renumbered C16 to C13, C18 to C14, C19 to C15, U10 to U11, U11 to U12
Changed lines of the file:
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@@
   (symbol (lib_id "Isolator:VO2611") (at 92.71 106.68 0) (unit 1)
     (in_bom yes) (on_board yes) (dnp no)
-    (property "Reference" "U10" (at 95.25 91.44 0)
+    (property "Reference" "U11" (at 95.25 91.44 0)
       (effects (font (size 1.27 1.27)) (justify left))
     )
@@
       (project "tms"
         (path "/dc88686f-c772-4c63-b1cc-83a281c6b46c/025e288f-ab42-4019-86f4-e6a324d46d8a"
-          (reference "U10") (unit 1)
+          (reference "U11") (unit 1)
         )
       )
@@
   (symbol (lib_id "Device:C") (at 144.78 85.09 90) (unit 1)
     (in_bom yes) (on_board yes) (dnp no)
-    (property "Reference" "C19" (at 144.78 78.74 90)
+    (property "Reference" "C15" (at 144.78 78.74 90)
       (effects (font (size 1.27 1.27)))
     )
@@
       (project "tms"
         (path "/dc88686f-c772-4c63-b1cc-83a281c6b46c/025e288f-ab42-4019-86f4-e6a324d46d8a"
-          (reference "C19") (unit 1)
+          (reference "C15") (unit 1)
         )
       )
@@
   (symbol (lib_id "Device:C") (at 144.78 73.66 90) (unit 1)
     (in_bom yes) (on_board yes) (dnp no)
-    (property "Reference" "C18" (at 144.78 67.31 90)
+    (property "Reference" "C14" (at 144.78 67.31 90)
       (effects (font (size 1.27 1.27)))
     )
@@
       (project "tms"
         (path "/dc88686f-c772-4c63-b1cc-83a281c6b46c/025e288f-ab42-4019-86f4-e6a324d46d8a"
-          (reference "C18") (unit 1)
+          (reference "C14") (unit 1)
         )
       )
@@
   (symbol (lib_id "Driver_FET:TC4422") (at 134.62 93.98 0) (unit 1)
     (in_bom yes) (on_board yes) (dnp no)
-    (property "Reference" "U11" (at 134.62 81.28 0)
+    (property "Reference" "U12" (at 134.62 81.28 0)
       (effects (font (size 1.27 1.27)))
     )
@@
       (project "tms"
         (path "/dc88686f-c772-4c63-b1cc-83a281c6b46c/025e288f-ab42-4019-86f4-e6a324d46d8a"
-          (reference "U11") (unit 1)
+          (reference "U12") (unit 1)
         )
       )
@@
   (symbol (lib_id "Device:C") (at 101.6 113.03 0) (unit 1)
     (in_bom yes) (on_board yes) (dnp no)
-    (property "Reference" "C16" (at 104.14 113.03 0)
+    (property "Reference" "C13" (at 104.14 113.03 0)
       (effects (font (size 1.27 1.27)) (justify left))
     )
@@
       (project "tms"
         (path "/dc88686f-c772-4c63-b1cc-83a281c6b46c/025e288f-ab42-4019-86f4-e6a324d46d8a"
-          (reference "C16") (unit 1)
-        )
-      )
+          (reference "C13") (unit 1)
+        )
+      )
