File: schematics/tms.kicad_sch (KiCad schematic)
At the start: 24 parts, among them J1 120V @ 60Hz, Q1 BT169B, SW1 SW_DIP_x01, SW2 SW_DIP_x01, SW3 SW_DIP_x01, U1 L7812CV, U2 L7805CV

Commit message: Small schematic fixes
Parts:
- removed C3: 0.22μF, symbol Device:C
- removed R7,R8,R9: 3x 10Ω, symbol Device:R
- A1: value Arduino_UNO_R3 -> Arduino_UNO_R4
- renumbered C4 to C3, C5 to C4, C6 to C5, C7 to C6, C8 to C7, C9 to C8, R10 to R7, R11 to R8, R12 to R9
Connections:
- net CHARGE CTRL: now also A1.19 (D4); no longer A1.17 (D2)
- net COMPARATOR STOP: now also A1.17 (D2); no longer A1.19 (D4)
Changed lines of the file:
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@@
   (junction (at 238.76 31.75) (diameter 0) (color 0 0 0 0)
   )
-  (junction (at 186.69 93.98) (diameter 0) (color 0 0 0 0)
-  )
   (junction (at 157.48 114.3) (diameter 0) (color 0 0 0 0)
   )
@@
     (stroke (width 0) (type default))
   )
-  (wire (pts (xy 204.47 93.98) (xy 203.2 93.98))
-    (stroke (width 0) (type default))
-  )
   (wire (pts (xy 186.69 93.98) (xy 186.69 104.14))
     (stroke (width 0) (type default))
@@
     (stroke (width 0) (type default))
   )
+  (wire (pts (xy 52.07 31.75) (xy 55.88 31.75))
+    (stroke (width 0) (type default))
+  )
+  (wire (pts (xy 210.82 107.95) (xy 198.12 107.95))
+    (stroke (width 0) (type default))
+  )
+  (wire (pts (xy 161.29 78.74) (xy 168.91 78.74))
+    (stroke (width 0) (type default))
+  )
+  (wire (pts (xy 170.18 105.41) (xy 170.18 104.14))
+    (stroke (width 0) (type default))
+  )
+  (wire (pts (xy 204.47 93.98) (xy 213.36 93.98))
+    (stroke (width 0) (type default))
+  )
   (wire (pts (xy 39.37 149.86) (xy 46.99 149.86))
     (stroke (width 0) (type default))
   )
-  (wire (pts (xy 52.07 31.75) (xy 55.88 31.75))
-    (stroke (width 0) (type default))
-  )
-  (wire (pts (xy 210.82 107.95) (xy 198.12 107.95))
-    (stroke (width 0) (type default))
-  )
-  (wire (pts (xy 161.29 78.74) (xy 168.91 78.74))
-    (stroke (width 0) (type default))
-  )
-  (wire (pts (xy 170.18 105.41) (xy 170.18 104.14))
-    (stroke (width 0) (type default))
-  )
-  (wire (pts (xy 204.47 93.98) (xy 213.36 93.98))
-    (stroke (width 0) (type default))
-  )
   (wire (pts (xy 157.48 93.98) (xy 186.69 93.98))
     (stroke (width 0) (type default))
@@
     (stroke (width 0) (type default))
   )
-  (wire (pts (xy 187.96 93.98) (xy 186.69 93.98))
-    (stroke (width 0) (type default))
-  )
   (wire (pts (xy 55.88 39.37) (xy 68.58 39.37))
     (stroke (width 0) (type default))
   )
+  (wire (pts (xy 39.37 154.94) (xy 46.99 154.94))
+    (stroke (width 0) (type default))
+  )
   (wire (pts (xy 148.59 96.52) (xy 157.48 96.52))
     (stroke (width 0) (type default))
@@
   )
   (wire (pts (xy 213.36 114.3) (xy 170.18 114.3))
-    (stroke (width 0) (type default))
-  )
-  (wire (pts (xy 39.37 154.94) (xy 46.99 154.94))
     (stroke (width 0) (type default))
   )
@@
     )
   )
-  (global_label "COMPARATOR STOP" (shape input) (at 39.37 154.94 180) (fields_autoplaced)
-    (effects (font (size 1.27 1.27)) (justify right))
-    (property "Intersheetrefs" "${INTERSHEET_REFS}" (at 18.3024 154.94 0)
+  (global_label "COMPARATOR STOP" (shape input) (at 39.37 149.86 180) (fields_autoplaced)
+    (effects (font (size 1.27 1.27)) (justify right))
+    (property "Intersheetrefs" "${INTERSHEET_REFS}" (at 18.3024 149.86 0)
       (effects (font (size 1.27 1.27)) (justify right) hide)
     )
@@
     )
   )
-  (global_label "CHARGE CTRL" (shape output) (at 39.37 149.86 180) (fields_autoplaced)
-    (effects (font (size 1.27 1.27)) (justify right))
-    (property "Intersheetrefs" "${INTERSHEET_REFS}" (at 23.5034 149.86 0)
+  (global_label "CHARGE CTRL" (shape output) (at 39.37 154.94 180) (fields_autoplaced)
+    (effects (font (size 1.27 1.27)) (justify right))
+    (property "Intersheetrefs" "${INTERSHEET_REFS}" (at 23.5034 154.94 0)
       (effects (font (size 1.27 1.27)) (justify right) hide)
     )
@@
     )
   )
-  (symbol (lib_id "Device:C") (at 191.77 93.98 90) (unit 1)
-    (in_bom yes) (on_board yes) (dnp no)
-    (property "Reference" "C3" (at 191.77 87.63 90)
-      (effects (font (size 1.27 1.27)))
-    )
-    (property "Value" "0.22μF" (at 191.77 90.17 90)
-      (effects (font (size 1.27 1.27)))
-    )
-    (property "Footprint" "" (at 195.58 93.0148 0)
-      (effects (font (size 1.27 1.27)) hide)
-    )
-    (property "Datasheet" "~" (at 191.77 93.98 0)
-      (effects (font (size 1.27 1.27)) hide)
-    )
-    (pin "1")
-    (pin "2")
-    (instances
-      (project "tms"
-        (path "/dc88686f-c772-4c63-b1cc-83a281c6b46c"
-          (reference "C3") (unit 1)
-        )
-      )
-    )
-  )
   (symbol (lib_id "Regulator_Linear:L7812") (at 229.87 31.75 0) (unit 1)
     (in_bom yes) (on_board yes) (dnp no) (fields_autoplaced)
@@
   (symbol (lib_id "Device:C") (at 238.76 35.56 0) (unit 1)
     (in_bom yes) (on_board yes) (dnp no)
-    (property "Reference" "C7" (at 242.57 34.29 0)
+    (property "Reference" "C6" (at 242.57 34.29 0)
       (effects (font (size 1.27 1.27)) (justify left))
     )
@@
       (project "tms"
         (path "/dc88686f-c772-4c63-b1cc-83a281c6b46c"
-          (reference "C7") (unit 1)
+          (reference "C6") (unit 1)
         )
       )
@@
   (symbol (lib_id "Device:R") (at 170.18 109.22 0) (mirror y) (unit 1)
     (in_bom yes) (on_board yes) (dnp no)
-    (property "Reference" "R10" (at 167.64 107.95 0)
+    (property "Reference" "R7" (at 167.64 107.95 0)
       (effects (font (size 1.27 1.27)) (justify left))
     )
@@
       (project "tms"
         (path "/dc88686f-c772-4c63-b1cc-83a281c6b46c"
-          (reference "R10") (unit 1)
+          (reference "R7") (unit 1)
         )
       )
@@
     )
   )
-  (symbol (lib_id "Device:R") (at 199.39 93.98 90) (unit 1)
-    (in_bom yes) (on_board yes) (dnp no)
-    (property "Reference" "R7,R8,R9" (at 199.39 87.63 90)
-      (effects (font (size 1.27 1.27)))
-    )
-    (property "Value" "3x 10Ω" (at 199.39 90.17 90)
-      (effects (font (size 1.27 1.27)))
-    )
-    (property "Footprint" "" (at 199.39 95.758 90)
-      (effects (font (size 1.27 1.27)) hide)
-    )
-    (property "Datasheet" "~" (at 199.39 93.98 0)
-      (effects (font (size 1.27 1.27)) hide)
-    )
-    (pin "1")
-    (pin "2")
-    (instances
-      (project "tms"
-        (path "/dc88686f-c772-4c63-b1cc-83a281c6b46c"
-          (reference "R7,R8,R9") (unit 1)
-        )
-      )
-    )
-  )
   (symbol (lib_id "Device:C") (at 220.98 35.56 0) (mirror y) (unit 1)
     (in_bom yes) (on_board yes) (dnp no)
-    (property "Reference" "C6" (at 217.17 34.29 0)
+    (property "Reference" "C5" (at 217.17 34.29 0)
       (effects (font (size 1.27 1.27)) (justify left))
     )
@@
       (project "tms"
         (path "/dc88686f-c772-4c63-b1cc-83a281c6b46c"
-          (reference "C6") (unit 1)
+          (reference "C5") (unit 1)
         )
       )
@@
   (symbol (lib_id "Device:C") (at 55.88 35.56 0) (unit 1)
     (in_bom yes) (on_board yes) (dnp no)
-    (property "Reference" "C4" (at 58.42 34.29 0)
+    (property "Reference" "C3" (at 58.42 34.29 0)
       (effects (font (size 1.27 1.27)) (justify left))
     )
@@
       (project "tms"
         (path "/dc88686f-c772-4c63-b1cc-83a281c6b46c"
-          (reference "C4") (unit 1)
+          (reference "C3") (unit 1)
         )
       )
@@
   (symbol (lib_id "Device:C") (at 238.76 58.42 0) (unit 1)
     (in_bom yes) (on_board yes) (dnp no)
-    (property "Reference" "C9" (at 242.57 57.15 0)
+    (property "Reference" "C8" (at 242.57 57.15 0)
       (effects (font (size 1.27 1.27)) (justify left))
     )
@@
       (project "tms"
         (path "/dc88686f-c772-4c63-b1cc-83a281c6b46c"
-          (reference "C9") (unit 1)
+          (reference "C8") (unit 1)
         )
       )
@@
   (symbol (lib_id "Device:R") (at 180.34 133.35 90) (unit 1)
     (in_bom yes) (on_board yes) (dnp no)
-    (property "Reference" "R12" (at 180.34 127 90)
+    (property "Reference" "R9" (at 180.34 127 90)
       (effects (font (size 1.27 1.27)))
     )
@@
       (project "tms"
         (path "/dc88686f-c772-4c63-b1cc-83a281c6b46c"
-          (reference "R12") (unit 1)
+          (reference "R9") (unit 1)
         )
       )
@@
   (symbol (lib_id "Device:C") (at 220.98 58.42 0) (mirror y) (unit 1)
     (in_bom yes) (on_board yes) (dnp no)
-    (property "Reference" "C8" (at 217.17 57.15 0)
+    (property "Reference" "C7" (at 217.17 57.15 0)
       (effects (font (size 1.27 1.27)) (justify left))
     )
@@
       (project "tms"
         (path "/dc88686f-c772-4c63-b1cc-83a281c6b46c"
-          (reference "C8") (unit 1)
+          (reference "C7") (unit 1)
         )
       )
@@
   (symbol (lib_id "Device:R") (at 172.72 133.35 90) (unit 1)
     (in_bom yes) (on_board yes) (dnp no)
-    (property "Reference" "R11" (at 172.72 127 90)
+    (property "Reference" "R8" (at 172.72 127 90)
       (effects (font (size 1.27 1.27)))
     )
@@
       (project "tms"
         (path "/dc88686f-c772-4c63-b1cc-83a281c6b46c"
-          (reference "R11") (unit 1)
+          (reference "R8") (unit 1)
         )
       )
@@
   (symbol (lib_id "Device:C") (at 68.58 35.56 0) (unit 1)
     (in_bom yes) (on_board yes) (dnp no)
-    (property "Reference" "C5" (at 71.12 34.29 0)
+    (property "Reference" "C4" (at 71.12 34.29 0)
       (effects (font (size 1.27 1.27)) (justify left))
     )
@@
       (project "tms"
         (path "/dc88686f-c772-4c63-b1cc-83a281c6b46c"
-          (reference "C5") (unit 1)
+          (reference "C4") (unit 1)
         )
       )
@@
       (effects (font (size 1.27 1.27)) (justify left))
     )
-    (property "Value" "Arduino_UNO_R3" (at 66.9641 134.62 0)
-      (effects (font (size 1.27 1.27)) (justify left))
-    )
+    (property "Value" "Arduino_UNO_R4" (at 66.9641 134.62 0)
+      (effects (font (size 1.27 1.27)) (justify left))
+    )
