File: schematics/charge.kicad_sch (KiCad schematic)
At the start: 56 parts, among them K1 AZ9861-1C-24DC2R1, Q2 NPN, Q3 NPN, T1 Transformer_1P_1S, U12 UA741, U3 VO2611, U4 VO2611, U5 UA741, U6 IL300, U7 UA741, U8 LM393, U9 VO2611

Commit message: Small schematic fixes
Parts:
- renumbered C12 to C11, C14 to C12, C21 to C9, R13 to R10, R14 to R11, R2 to R12, R19 to R13, R1 to R14, R3 to R15, R15 to R16, R16 to R17, R17 to R18, R18 to R19, R25 to R20, R26 to R21, R27 to R22, R22 to R23, R20 to R24, R21 to R25, R23 to R26, R24 to R27, U12 to U10

Commit message: Schematic update
Parts:
- removed F1: Fuse, symbol Device:Fuse
Changed lines of the file:
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@@
+    (stroke (width 0) (type default))
+  )
+  (wire (pts (xy 187.96 36.83) (xy 187.96 46.99))
     (stroke (width 0) (type default))
   )
@@
     (stroke (width 0) (type default))
   )
-  (wire (pts (xy 187.96 45.72) (xy 187.96 46.99))
-    (stroke (width 0) (type default))
-  )
   (wire (pts (xy 205.74 46.99) (xy 228.6 46.99))
     (stroke (width 0) (type default))
@@
   )
   (wire (pts (xy 29.21 163.83) (xy 31.75 163.83))
-    (stroke (width 0) (type default))
-  )
-  (wire (pts (xy 187.96 36.83) (xy 187.96 38.1))
     (stroke (width 0) (type default))
   )
@@
         )
       )
-    )
-  )
-  (symbol (lib_id "Device:Fuse") (at 187.96 41.91 0) (unit 1)
-    (in_bom yes) (on_board yes) (dnp no) (fields_autoplaced)
-    (property "Reference" "F1" (at 190.5 40.64 0)
-      (effects (font (size 1.27 1.27)) (justify left))
-    )
-    (property "Value" "Fuse" (at 190.5 43.18 0)
-      (effects (font (size 1.27 1.27)) (justify left))
-    )
-    (property "Footprint" "" (at 186.182 41.91 90)
-      (effects (font (size 1.27 1.27)) hide)
-    )
-    (property "Datasheet" "~" (at 187.96 41.91 0)
-      (effects (font (size 1.27 1.27)) hide)
-    )
-    (pin "1")
-    (pin "2")
-    (instances
-      (project "tms"
-        (path "/dc88686f-c772-4c63-b1cc-83a281c6b46c/52808854-7c95-4ac8-9e37-1a1e5d6f75e2"
-          (reference "F1") (unit 1)
-        )
-      )
